File: pcb/RedFly-Shield_v14.sch (EAGLE design)
At the start: 66 parts, among them IC1 74LVC244, U1 TS1117-3.3V, X1 PASSER, X2 PASSER, X3 PASSER, X4 PASSER

Commit message: updated license infos
Other:
- note added: "Released under the Creative Commons Attribution Share-Alike License"
- note added: "http://creativecommons.org/licenses/by-sa/4.0/"
- note removed: "Released under the Creative Commons Attribution Share-Alike 3.0 License"
- note removed: "http://creativecommons.org/licenses/by-sa/3.0/"
Changed lines of the file:
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@@
 <?xml version="1.0" encoding="utf-8"?>
 <!DOCTYPE eagle SYSTEM "eagle.dtd">
-<eagle version="6.4">
+<eagle version="6.5.0">
 <drawing>
 <settings>
@@
 <setting verticaltext="up"/>
 </settings>
-<grid distance="0.05" unitdist="inch" unit="inch" style="lines" multiple="1" display="yes" altdistance="0.025" altunitdist="inch" altunit="inch"/>
+<grid distance="0.1" unitdist="inch" unit="inch" style="lines" multiple="1" display="no" altdistance="0.01" altunitdist="inch" altunit="inch"/>
 <layers>
 <layer number="1" name="Top" color="4" fill="1" visible="no" active="no"/>
@@
 <wire x1="72.39" y1="71.12" x2="75.057" y2="71.12" width="0.8128" layer="94"/>
 <wire x1="114.3" y1="71.12" x2="116.967" y2="71.12" width="0.8128" layer="94"/>
-<text x="161.29" y="31.75" size="1.27" layer="95">Released under the Creative Commons Attribution Share-Alike 3.0 License</text>
-<text x="161.29" y="29.21" size="1.27" layer="95">http://creativecommons.org/licenses/by-sa/3.0/</text>
+<text x="161.29" y="31.75" size="1.27" layer="95">Released under the Creative Commons Attribution Share-Alike License</text>
+<text x="161.29" y="29.21" size="1.27" layer="95">http://creativecommons.org/licenses/by-sa/4.0/</text>
 <text x="161.29" y="25.4" size="1.27" layer="95">Designed by Andreas Watterott (Watterott electronic)</text>
 <text x="52.07" y="166.37" size="3.81" layer="250">Arduino</text>
