File: pcb/RedFly-Shield_v14.sch (EAGLE design)
At the start: 66 parts, among them IC1 74LVC244, U1 TS1117-3.3V, X1 PASSER, X2 PASSER, X3 PASSER, X4 PASSER

Commit message: cleaned up schematics and layout
Changed lines of the file:
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@@
 <setting verticaltext="up"/>
 </settings>
-<grid distance="0.1" unitdist="inch" unit="inch" style="lines" multiple="1" display="no" altdistance="0.01" altunitdist="inch" altunit="inch"/>
+<grid distance="0.05" unitdist="inch" unit="inch" style="lines" multiple="1" display="yes" altdistance="0.025" altunitdist="inch" altunit="inch"/>
 <layers>
 <layer number="1" name="Top" color="4" fill="1" visible="no" active="no"/>
@@
 <part name="C7" library="rcl" deviceset="C-EU" device="C0603" value="100nF"/>
 <part name="C8" library="rcl" deviceset="C-EU" device="C0603" value="2uF"/>
-<part name="FRAME1" library="frames" deviceset="A4L-LOC" device=""/>
 <part name="IC1" library="74xx-eu" deviceset="74*244" device="DW" technology="HC" value="74LVC244"/>
 <part name="GND10" library="supply1" deviceset="GND" device=""/>
@@
 <part name="GND." library="wirepad" deviceset="WIREPAD" device="1,6/0,8"/>
 <part name="GND3" library="supply1" deviceset="GND" device=""/>
+<part name="FRAME1" library="we-symbol" deviceset="FRAME-A4L" device=""/>
 </parts>
 <sheets>
@@
 <wire x1="72.39" y1="71.12" x2="75.057" y2="71.12" width="0.8128" layer="94"/>
 <wire x1="114.3" y1="71.12" x2="116.967" y2="71.12" width="0.8128" layer="94"/>
-<text x="161.29" y="31.75" size="1.27" layer="95">Released under the Creative Commons Attribution Share-Alike License</text>
-<text x="161.29" y="29.21" size="1.27" layer="95">http://creativecommons.org/licenses/by-sa/4.0/</text>
-<text x="161.29" y="25.4" size="1.27" layer="95">Designed by Andreas Watterott (Watterott electronic)</text>
+<text x="162.56" y="21.59" size="1.27" layer="95">Released under the Creative Commons Attribution Share-Alike License</text>
+<text x="162.56" y="19.05" size="1.27" layer="95">http://creativecommons.org/licenses/by-sa/4.0/</text>
+<text x="162.56" y="15.24" size="1.27" layer="95">Designed by Andreas Watterott (Watterott electronic)</text>
 <text x="52.07" y="166.37" size="3.81" layer="250">Arduino</text>
 <text x="46.99" y="74.93" size="3.81" layer="250">Level Converter</text>
@@
 <attribute name="VALUE" x="160.782" y="96.266" size="1.778" layer="96"/>
 </instance>
-<instance part="FRAME1" gate="G$1" x="0" y="0" smashed="yes">
-<attribute name="DRAWING_NAME" x="217.17" y="15.24" size="2.54" layer="94" font="vector"/>
-<attribute name="LAST_DATE_TIME" x="217.17" y="10.16" size="2.286" layer="94" font="vector"/>
-<attribute name="SHEET" x="230.505" y="5.08" size="2.54" layer="94" font="vector"/>
-</instance>
 <instance part="IC1" gate="A" x="34.29" y="54.61" smashed="yes" rot="MR0">
 <attribute name="NAME" x="41.91" y="62.865" size="1.778" layer="95" rot="MR0"/>
@@
 <attribute name="VALUE" x="109.22" y="144.78" size="1.778" layer="96" rot="R90"/>
 </instance>
-<instance part="X1" gate="G$1" x="166.37" y="19.05"/>
-<instance part="X2" gate="G$1" x="173.99" y="19.05"/>
-<instance part="X3" gate="G$1" x="181.61" y="19.05"/>
-<instance part="X4" gate="G$1" x="189.23" y="19.05"/>
-<instance part="LOGO1" gate="G$1" x="201.93" y="19.05"/>
+<instance part="X1" gate="G$1" x="165.1" y="7.62" smashed="yes"/>
+<instance part="X2" gate="G$1" x="170.18" y="7.62" smashed="yes"/>
+<instance part="X3" gate="G$1" x="175.26" y="7.62" smashed="yes"/>
+<instance part="X4" gate="G$1" x="180.34" y="7.62" smashed="yes"/>
+<instance part="LOGO1" gate="G$1" x="208.28" y="7.62"/>
 <instance part="WIFI-WLAN" gate="G$1" x="198.12" y="116.84" smashed="yes">
 <attribute name="NAME" x="180.34" y="150.368" size="1.778" layer="95"/>
@@
 <attribute name="VALUE" x="240.03" y="144.78" size="1.778" layer="96" rot="R90"/>
 </instance>
-<instance part="LOGO2" gate="G$1" x="201.93" y="11.43"/>
+<instance part="LOGO2" gate="G$1" x="198.12" y="7.62"/>
 <instance part="ARD" gate="G$1" x="62.23" y="124.46"/>
 <instance part="RESET" gate="G$1" x="96.52" y="149.86" rot="R270"/>
@@
 <attribute name="VALUE" x="31.75" y="123.19" size="1.778" layer="96" rot="R270"/>
 </instance>
+<instance part="FRAME1" gate="G$1" x="0" y="0"/>
 </instances>
 <busses>
